Commit message: [DRAGON][URDF] Add DJI camera model, create new xacro under dragon v1.5, and update bringup.launch for battery and model suffix

File: robots/dragon/urdf/v1_5/dragon_common.xacro (robot description, xacro)
@@ -33,5 +33,5 @@
     </visual>
   </xacro:macro>
-  <xacro:macro name="extra_module" params="name parent *origin *inertial visible:=0 model_url:=1 scale:=1">
+  <xacro:macro name="extra_module" params="name parent *origin *inertial visible:=0 model_url:=1 scale:=1 visual_x:=0 visual_y:=0 visual_z:=0 visual_roll:=0 visual_pitch:=0 visual_yaw:=0">
     <joint name="${parent}2${name}" type="fixed">
       <parent link="${parent}"/>
@@ -43,5 +43,5 @@
       <xacro:if value="${visible == 1}">
         <visual>
-          <origin rpy="0 0 0" xyz="0 0 0"/>
+          <origin rpy="${visual_roll} ${visual_pitch} ${visual_yaw}" xyz="${visual_x} ${visual_y} ${visual_z}"/>
           <geometry>
             <mesh filename="${model_url}" scale= "${scale} ${scale} ${scale}"/>
