Commit message: [DRAGON][URDF] Fix v1.5 collision geometry to improve body, joint, and ducted fan coverage

File: robots/dragon/urdf/v1_5/dragon_common.xacro (robot description, xacro)
@@ -14,4 +14,10 @@
   <xacro:property name="gimbal_roll_x_offset" value="-0.0065" />
   <xacro:property name="gimbal_pitch_z_offset" value="0.0265" />
+  <!-- collision geometry [m] -->
+  <xacro:property name="link_collision_length" value="0.60" />
+  <xacro:property name="link_collision_width" value="0.13" />
+  <xacro:property name="link_collision_height" value="0.19" />
+  <xacro:property name="link_collision_y_offset" value="-0.017" />
+  <xacro:property name="link_collision_z_offset" value="0.005" />
   <!-- dynamics -->
   <m_f_rate value="0" /> <!-- drug torque rate -->
@@ -21,7 +27,7 @@
     <!-- box collision geometry does not work well for FCL -->
     <collision>
-    <origin rpy="0 0 0" xyz="${link_length* 0.5} 0 0"/>
+    <origin rpy="0 0 0" xyz="${link_length* 0.5} ${link_collision_y_offset} ${link_collision_z_offset}"/>
     <geometry>
-    <box size="${link_length} 0.15 0.1686"/>
+    <box size="${link_collision_length} ${link_collision_width} ${link_collision_height}"/>
     </geometry>
     </collision>

File: robots/dragon/urdf/v1_5/dragon_link.urdf.xacro (robot description, xacro)
@@ -83,5 +83,5 @@
         <origin rpy="${pi/2} 0 0" xyz="0 0 0.02"/>
         <geometry>
-          <cylinder length="0.3" radius="0.09" />
+          <cylinder length="0.40" radius="0.09" />
         </geometry>
       </collision>
