Commit message: [DRAGON][URDF] Add MID360 optical origin frame (lidar_origin) to  robot models

File: robots/dragon/robots/quad/v1_5_202601.urdf.xacro (robot description, xacro)
@@ -30,3 +30,16 @@
     </inertial>
   </xacro:extra_module>
+  <!-- MID360 optical origin: the physical ray origin of the published clouds.
+       lidar_imu sits at (0.011, 0.02329, -0.04412) from here, which is the
+       MID360 IMU-to-optical extrinsic FAST-LIO carries as mapping/extrinsic_T. -->
+  <xacro:extra_module name = "lidar_origin" parent = "livox_mid360" visible = "0" >
+    <origin xyz="0 0 ${-0.02592 + 0.047}" rpy="0 0 0"/>
+    <inertial>
+      <origin xyz="0 0 0" rpy="0 0 0"/>
+      <mass value="0"/>
+      <inertia
+          ixx="0.0" iyy="0.0" izz="0.0"
+          ixy="0.0" ixz="0.0" iyz="0.0"/>
+    </inertial>
+  </xacro:extra_module>
 </robot>

File: robots/dragon/robots/quad/v1_5_202601_dji_on.urdf.xacro (robot description, xacro)
@@ -32,3 +32,16 @@
     </inertial>
   </xacro:extra_module>
+  <!-- MID360 optical origin: the physical ray origin of the published clouds.
+       lidar_imu sits at (0.011, 0.02329, -0.04412) from here, which is the
+       MID360 IMU-to-optical extrinsic FAST-LIO carries as mapping/extrinsic_T. -->
+  <xacro:extra_module name = "lidar_origin" parent = "livox_mid360" visible = "0" >
+    <origin xyz="0 0 ${-0.02592 + 0.047}" rpy="0 0 0"/>
+    <inertial>
+      <origin xyz="0 0 0" rpy="0 0 0"/>
+      <mass value="0"/>
+      <inertia
+          ixx="0.0" iyy="0.0" izz="0.0"
+          ixy="0.0" ixz="0.0" iyz="0.0"/>
+    </inertial>
+  </xacro:extra_module>
 </robot>

File: robots/dragon/robots/quad/v1_5_202601_dji_on_no_bat.urdf.xacro (robot description, xacro)
@@ -33,3 +33,16 @@
     </inertial>
   </xacro:extra_module>
+  <!-- MID360 optical origin: the physical ray origin of the published clouds.
+       lidar_imu sits at (0.011, 0.02329, -0.04412) from here, which is the
+       MID360 IMU-to-optical extrinsic FAST-LIO carries as mapping/extrinsic_T. -->
+  <xacro:extra_module name = "lidar_origin" parent = "livox_mid360" visible = "0" >
+    <origin xyz="0 0 ${-0.02592 + 0.047}" rpy="0 0 0"/>
+    <inertial>
+      <origin xyz="0 0 0" rpy="0 0 0"/>
+      <mass value="0"/>
+      <inertia
+          ixx="0.0" iyy="0.0" izz="0.0"
+          ixy="0.0" ixz="0.0" iyz="0.0"/>
+    </inertial>
+  </xacro:extra_module>
 </robot>

File: robots/dragon/robots/quad/v1_5_202601_no_bat.urdf.xacro (robot description, xacro)
@@ -31,3 +31,16 @@
     </inertial>
   </xacro:extra_module>
+  <!-- MID360 optical origin: the physical ray origin of the published clouds.
+       lidar_imu sits at (0.011, 0.02329, -0.04412) from here, which is the
+       MID360 IMU-to-optical extrinsic FAST-LIO carries as mapping/extrinsic_T. -->
+  <xacro:extra_module name = "lidar_origin" parent = "livox_mid360" visible = "0" >
+    <origin xyz="0 0 ${-0.02592 + 0.047}" rpy="0 0 0"/>
+    <inertial>
+      <origin xyz="0 0 0" rpy="0 0 0"/>
+      <mass value="0"/>
+      <inertia
+          ixx="0.0" iyy="0.0" izz="0.0"
+          ixy="0.0" ixz="0.0" iyz="0.0"/>
+    </inertial>
+  </xacro:extra_module>
 </robot>

File: robots/dragon/robots/quad/vim4_202311.urdf.xacro (robot description, xacro)
@@ -31,3 +31,16 @@
     </inertial>
   </xacro:extra_module>
+  <!-- MID360 optical origin: the physical ray origin of the published clouds.
+       lidar_imu sits at (0.011, 0.02329, -0.04412) from here, which is the
+       MID360 IMU-to-optical extrinsic FAST-LIO carries as mapping/extrinsic_T. -->
+  <xacro:extra_module name = "lidar_origin" parent = "livox_mid360" visible = "0" >
+    <origin xyz="0 0 ${-0.02592 + 0.047}" rpy="0 0 0"/>
+    <inertial>
+      <origin xyz="0 0 0" rpy="0 0 0"/>
+      <mass value="0"/>
+      <inertia
+          ixx="0.0" iyy="0.0" izz="0.0"
+          ixy="0.0" ixz="0.0" iyz="0.0"/>
+    </inertial>
+  </xacro:extra_module>
 </robot>
